File: Hardware/MicroMod-Ethernet-Function-Board.sch (EAGLE design)
At the start: 69 parts, among them J1 MAGJACK_SYM, J11 MICROMOD_STANDARD, Q5 20V/4.2A/52mΩ/1.4W, Q6 600mA/40V, U1 EEPROM, U2 AG980X, U3 W5500-ETHERNET, U4 3.3V, Y1 24MHz

Commit message: Update PoE module to DP990X.
Parts:
- removed PWR_LED: JUMPER-SMT_2_NC_TRACE_SILK, SparkFun-Jumpers:JUMPER-SMT_2_NC_TRACE_SILK
- removed Q6: 600mA/40V, SparkFun-DiscreteSemi:TRANS_PNP-MMBT4403
- removed U2: AG980X, Ethernet:AG980X
- added C25, C26: 10uF, SparkFun-Capacitors:10UF-0805-25V-10%
- added C8: 100uF, SparkFun-Capacitors:100UF-POLAR-25V-20%(ELEC)
- added ISO1, ISO2: JUMPER-COMBO_2_NC_TRACE, SparkFun-Jumpers:JUMPER-COMBO_2_NC_TRACE
- added JP5: JUMPER-SMT_2_NO_SILK, SparkFun-Jumpers:JUMPER-SMT_2_NO_SILK
- added L1: 2.2uH, SparkFun-Coils:INDUCTOR-0805_WIDE-2.2UH
- added LOAD, POE_LED: JUMPER-SMT_2_NC_TRACE_SILK, SparkFun-Jumpers:JUMPER-SMT_2_NC_TRACE_SILK
- added Q1: 220mA/50V/3.5Ω, SparkFun-DiscreteSemi:MOSFET-NCH-BSS138
- added R22: 10k, SparkFun-Resistors:10KOHM-0603-1/10W-1%
- added U5: POE_PSU-DP990X, Ethernet:POE_PSU-DP990X
- C13: value 0.22uF -> 1.0uF; device SparkFun-Capacitors:0.22UF-0603-25V-10% -> SparkFun-Capacitors:1.0UF-0603-16V-10%
- C19: value 22uF -> 1nF; device SparkFun-Capacitors:22UF-1206-50V-10% -> SparkFun-Capacitors:1.0NF/1000PF-1206-2KV-10%
- C21, C22: value 10nF -> 6.8nF; device SparkFun-Capacitors:10NF-0603-50V-10% -> SparkFun-Capacitors:6.8NF/6800PF-0603-50V-5%
- C7: value 560uF/25V -> 10uF; device SparkFun-Capacitors:560UF-PANASONIC_G-25V-20% -> SparkFun-Capacitors:10UF-0805-25V-10%
- JP4: device SparkFun-Jumpers:JUMPER-SMT_2_NO_SILK -> SparkFun-Jumpers:JUMPER-SMT_2_NC_TRACE_SILK
- R13, R18, R19, R20: value 47 -> 49.9; device SparkFun-Resistors:47OHM-0603-1/10W-1% -> SparkFun-Resistors:49.9OHM-0603-1/10W-1%
- R2: value 470 -> 510; device SparkFun-Resistors:470OHM-0603-1/10W-1% -> SparkFun-Resistors:510OHM-2010-1/2W-5%
- R6, R7: value 100k -> 10k; device SparkFun-Resistors:100KOHM-0603-1/10W-1% -> SparkFun-Resistors:10KOHM-0603-1/10W-1%
- R8: value 12.1k -> 12.4k; device SparkFun-Resistors:12.1KOHM-0603-1/10W-1% -> SparkFun-Resistors:12.4KOHM-0603-1/10W-1%
- U3: value W5500-ETHERNET -> W5500; device Ethernet:W5500-ETHERNET -> SparkFun-IC-Comms:W5500
- Y1: value 24MHz -> 25MHz; device SparkFun-Clocks:CRYSTAL-24MHZ-SMD-2.0X1.6MM -> SparkFun-Clocks:CRYSTAL-25MHZ-SMD-2.0X1.6MM
Connections:
- removed net N$4: J11.PWR_EN, R2.2
- new net 5V_FILTER: C26.1, D1.A, L1.2, LOAD.2, POE_LED.2
- new net N$12: JP5.2, R22.2, U1.WP
- new net N$14: ISO1.2, U5.VIN+
- new net N$18: ISO2.2, U5.VIN-
- new net N$9: LOAD.1, R2.2
- net 3.3V: now also R22.1
- net 5V: no longer PWR_LED.2
- net 5V_RAW: now also C25.1, C7.1, C8.+, L1.1, U5.VDC+; no longer C7.+, D1.A, U2.VDC+
- net GND: now also C25.2, C26.2, C7.2, C8.-, JP5.1, Q1.S, R2.1, U5.VDC-; no longer C7.-, R7.1, U1.WP, U2.VDC-
- net N$11: now also Q1.D, R7.1; no longer Q6.C, R7.2
- net N$6: now also POE_LED.1; no longer PWR_LED.1
- net PW+: now also ISO1.1; no longer U2.VIN+
- net PW-: now also ISO2.1; no longer U2.VIN-
- net PWR_EN: now also J11.PWR_EN, Q1.G; no longer Q6.B, R2.1
- net VCC_IN: now also R7.2; no longer Q6.E
Other:
- note added: "Dummy Load: 100mA"
- note added: "Fix WP on eeprom"
- note added: "Fix power control"
- note added: "Replace load R with 50 Ohm"
- note removed: "Replace 10nF caps with 6.8nF caps"
- note removed: "Replace 12.1k with new 12.4k"
- note removed: "Replace 22uF with 1nF/2kV 1206 cap"
- note removed: "Replace 24MHz with new 25MHz"
- note removed: "Replace 47 Ohm res with 49.9"
- moved on the sheet: C13, C24, C3, C4, D1, D5, MEAS, Q5, R11, R2, R6, R7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

Commit message: Add x01 panel files
Parts:
- added LED1, LED2: JUMPER-SMT_2_NC_TRACE_SILK, SparkFun-Jumpers:JUMPER-SMT_2_NC_TRACE_SILK
- added R23, R24, R30, R4: 10k, SparkFun-Resistors:10KOHM-0603-1/10W-1%
- R3, R5: value 330 -> 1k; device SparkFun-Resistors:330OHM-0603-1/10W-1% -> SparkFun-Resistors:1KOHM-0603-1/10W-1%
Connections:
- new net N$17: R30.2, U3.RSVD23
- new net N$3: J1.GRN-, LED2.1
- new net N$4: J1.YLW-, LED1.1
- net 3.3V: now also R23.2, R24.2, R4.2
- net ACT_LED: now also LED2.2; no longer J1.GRN-
- net ETH_!CS!: now also R23.1
- net ETH_!INT!: now also R4.1
- net ETH_!RST!: now also R24.1
- net GND: now also R30.1
- net LINK_LED: now also LED1.2; no longer J1.YLW-
Other:
- note added: "Default: PMODE 111 10/100 Auto-Negotiate"
- note removed: "Default: PMODE 111 - 10/100 Auto-Negotiate"
- note removed: "Fix WP on eeprom"
- moved on the sheet: C1, C10, C11, C12, C14, C15, C16, C17, C18, C2, C20, C21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

Commit message: Update PROD_IDs
Parts:
- J1: value MAGJACK_SYM -> MAGJACK-POE; device Ethernet:MAGJACK_SYM -> SparkFun-Connectors:MAGJACK-POE
- R2: value 510 -> 49.9 1/2W; device SparkFun-Resistors:510OHM-2010-1/2W-5% -> SparkFun-Resistors:49.9OHM-1206-1/2W-1%
- U5: device Ethernet:POE_PSU-DP990X -> SparkFun-IC-Power:POE_PSU-DP990X
Other:
- note removed: "Fix power control"
Changed lines of the file:
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@@
 <part name="LOGO2" library="SparkFun-Aesthetics" deviceset="SPECIAL_INSTRUCTIONS" device="-ORDERING"/>
 <part name="U3" library="SparkFun-IC-Comms" deviceset="W5500" device=""/>
-<part name="J1" library="Ethernet" deviceset="MAGJACK_SYM" device=""/>
+<part name="J1" library="SparkFun-Connectors" deviceset="MAGJACK-POE" device=""/>
 <part name="Y1" library="SparkFun-Clocks" deviceset="CRYSTAL-25MHZ" device="-SMD-2.0X1.6MM" value="25MHz"/>
 <part name="C5" library="SparkFun-Capacitors" deviceset="10PF" device="-0603-50V-5%" value="10pF"/>
@@
 <part name="GND5" library="SparkFun-PowerSymbols" deviceset="GND" device=""/>
 <part name="U$4" library="SparkFun-PowerSymbols" deviceset="VCCA" device=""/>
-<part name="U5" library="Ethernet" deviceset="POE_PSU" device="-DP990X" value="POE_PSU-DP990X"/>
+<part name="U5" library="SparkFun-IC-Power" deviceset="POE_PSU" device="-DP990X" value="POE_PSU-DP990X"/>
 <part name="C8" library="SparkFun-Capacitors" deviceset="100UF-POLAR" device="-25V-20%(ELEC)" value="100uF"/>
 <part name="C7" library="SparkFun-Capacitors" deviceset="10UF" device="-0805-25V-10%" value="10uF"/>
@@
 <part name="JP5" library="SparkFun-Jumpers" deviceset="JUMPER-SMT_2_NO" device="_SILK" package3d_urn="urn:adsk.eagle:package:39279/1"/>
 <part name="Q1" library="SparkFun-DiscreteSemi" deviceset="MOSFET-NCH" device="-BSS138" value="220mA/50V/3.5Ω"/>
-<part name="R2" library="SparkFun-Resistors" deviceset="510OHM" device="-2010-1/2W-5%" value="510"/>
+<part name="R2" library="SparkFun-Resistors" deviceset="49.9OHM" device="-1206-1/2W-1%" value="49.9 1/2W"/>
 <part name="LED1" library="SparkFun-Jumpers" deviceset="JUMPER-SMT_2_NC_TRACE" device="_SILK" package3d_urn="urn:adsk.eagle:package:39281/1" value="JUMPER-SMT_2_NC_TRACE_SILK"/>
 <part name="LED2" library="SparkFun-Jumpers" deviceset="JUMPER-SMT_2_NC_TRACE" device="_SILK" package3d_urn="urn:adsk.eagle:package:39281/1" value="JUMPER-SMT_2_NC_TRACE_SILK"/>
@@
 <wire x1="180.34" y1="137.16" x2="0" y2="137.16" width="0.2032" layer="97" style="longdash"/>
 <wire x1="330.2" y1="137.16" x2="330.2" y2="279.4" width="0.2032" layer="97" style="longdash"/>
-<text x="53.34" y="287.02" size="1.27" layer="91">Fix power control</text>
 <text x="53.34" y="284.48" size="1.27" layer="91">Replace load R with 50 Ohm</text>
 <text x="236.22" y="71.12" size="1.778" layer="97" font="vector" align="center">Dummy Load: 100mA</text>
@@
 <attribute name="VALUE" x="309.88" y="81.28" size="1.778" layer="96" font="vector"/>
 </instance>
-<instance part="R2" gate="G$1" x="243.84" y="88.9" smashed="yes" rot="R90">
+<instance part="R2" gate="R1" x="243.84" y="88.9" smashed="yes" rot="R90">
 <attribute name="NAME" x="242.316" y="88.9" size="1.778" layer="95" font="vector" rot="R90" align="bottom-center"/>
 <attribute name="VALUE" x="245.364" y="88.9" size="1.778" layer="96" font="vector" rot="R90" align="top-center"/>
@@
 <pinref part="GND31" gate="1" pin="GND"/>
 <wire x1="243.84" y1="81.28" x2="243.84" y2="83.82" width="0.1524" layer="91"/>
-<pinref part="R2" gate="G$1" pin="1"/>
+<pinref part="R2" gate="R1" pin="1"/>
 </segment>
 <segment>
@@
 <pinref part="LOAD" gate="G$1" pin="1"/>
 <wire x1="243.84" y1="93.98" x2="243.84" y2="96.52" width="0.1524" layer="91"/>
-<pinref part="R2" gate="G$1" pin="2"/>
-</segment>
-</net>
+<pinref part="R2" gate="R1" pin="2"/>
+</segment>
+</net>

Commit message: Connect PWR LED to 3.3V rail. Add POE LED. Add pin 1 indicator to PoE module. Add hot caution.
Parts:
- added D2: RED, SparkFun-LED:LED-RED0603
- added PWR_LED: JUMPER-SMT_2_NC_TRACE_SILK, SparkFun-Jumpers:JUMPER-SMT_2_NC_TRACE_SILK
- added R25: 1k, SparkFun-Resistors:1KOHM-0603-1/10W-1%
- D5: value RED -> Yellow; device SparkFun-LED:LED-RED0603 -> SparkFun-LED:LED-YELLOW0603
Connections:
- removed net N$12: JP5.2, R22.2, U1.WP
- new net EWP: J11.EEPROM_WP, JP5.2, R22.2, U1.WP
- new net N$19: PWR_LED.1, R25.2
- new net N$20: D2.A, R25.1
- net 3.3V: now also PWR_LED.2
- net GND: now also D2.C
Other:
- note added: "Add EEPROM WP connection"
- note added: "v10"
- note removed: "Replace load R with 50 Ohm"
- note removed: "x01"
- moved on the sheet: C4, JP5, R22, U1

Commit message: Add ESD to TX/RX, landmarks to PoE module, additional GND thermals.
Parts:
- added D7: DT1042-04SO, SparkFun-DiscreteSemi:TVS_DIODE_ARRAYSMD
- added TP1: TEST-POINT3X4, SparkFun-Connectors:TEST-POINT3X4
- POE: value PoE System -> JUMPER-SMT_2_NC_TRACE_SILK
- renumbered JP4 to POE
Connections:
- net N$14 renamed PW1+
- net N$18 renamed PW1-
- net 3.3V: now also TP1.1
- net GND-ISO: now also D7.VSS
- net RD+: now also D7.IO2
- net RD-: now also D7.IO3
- net TD+: now also D7.IO1
- net TD-: now also D7.IO4
Other:
- note added: "v11"
- note removed: "Add EEPROM WP connection"
- note removed: "v10"
- moved on the sheet: C13, C20, C21, C22, C23, C24, C3, MEAS, R13, R14, R15, R16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
